File: Board/ShifterBit.brd (EAGLE design)
At the start: 27.2 x 61 mm, 13 parts

Commit message: fixed missing connection
Connections:
- removed net VBAT: P1.9
- net VCC: now also P1.9
Changed lines of the file:
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@@
 <wire x1="15.6464" y1="15.4432" x2="23.9776" y2="15.4432" width="0.2032" layer="16"/>
 <wire x1="15.8496" y1="66.4464" x2="15.75" y2="66.635" width="0.2032" layer="16"/>
+<contactref element="P1" pad="9"/>
+<wire x1="3.1" y1="14.11" x2="11.495" y2="20.3838" width="0" layer="19" extent="16-16"/>
 </signal>
 <signal name="SIG_OUT">
@@
 <wire x1="3.2512" y1="19.304" x2="3.1" y2="19.19" width="0.2032" layer="16"/>
 </signal>
-<signal name="VBAT">
-<contactref element="P1" pad="9"/>
-</signal>
 <signal name="D5">
